Commit message: Changes made to port with bot, not working!

File: description/robot.urdf.xacro (robot description, xacro)
@@ -2,4 +2,6 @@
 <robot xmlns:xacro="http://www.ros.org/wiki/xacro"  name="robot">
     <xacro:include filename="robot_core.xacro"/>
-    <xacro:include filename="gazebo_control.xacro"/>
+    <!-- <xacro:include filename="ros2_control.xacro"/> -->
+    <xacro:include filename="roboclaw_ros2_control.xacro"/>
+    <!-- <xacro:include filename="gazebo_control.xacro"/> -->
 </robot>

File: description/robot_core.xacro (robot description, xacro)
@@ -86,5 +86,5 @@
                 <cylinder length="${wheel_link_length}" radius="${wheel_link_radius}"/>
             </geometry>
-            <material name="black" />
+            <material name="blue" />
         </visual>
         <collision>
