Commit message: Updates to roboclaw

File: description/roboclaw_ros2_control.xacro (robot description, xacro)
@@ -10,5 +10,5 @@
     <state_interface name="position"/>
     <param name="address">128</param>
-    <param name="qppr">500</param>
+    <param name="qppr">35</param>
     <param name="motor_type">M2</param>
   </joint>
@@ -17,5 +17,5 @@
     <state_interface name="position"/>
     <param name="address">128</param>
-    <param name="qppr">500</param>
+    <param name="qppr">35</param>
     <param name="motor_type">M1</param>
     <!-- Add other configurations as necessary -->

File: description/robot.urdf.xacro (robot description, xacro)
@@ -3,5 +3,6 @@
     <xacro:include filename="robot_core.xacro"/>
     <!-- <xacro:include filename="ros2_control.xacro"/> -->
-    <xacro:include filename="roboclaw_ros2_control.xacro"/>
-    <!-- <xacro:include filename="gazebo_control.xacro"/> -->
+    <!-- <xacro:include filename="roboclaw_ros2_control.xacro"/> -->
+    <xacro:include filename="gazebo_control.xacro"/>
+    <xacro:include filename="lidar.xacro"/>
 </robot>

File: description/robot_core.xacro (robot description, xacro)
@@ -43,4 +43,10 @@
     <link name="dummy">
     </link>
+    <joint name="base_footprint_joint" type="fixed">
+        <parent link="dummy" />
+        <child link="base_footprint" />
+        <origin xyz ="0 0 0" rpy="0 0 0"/>
+    </joint>
+    <link name="base_footprint"></link>
     <joint name="body_joint" type="fixed">
         <parent link="dummy" />
