Commit message: Robot Not moving left or Right

File: description/diff_dr_gaz.xacro (robot description, xacro)
@@ -42,5 +42,5 @@
             <max_wheel_acceleration>10.0</max_wheel_acceleration>
             <odometry_frame>odom</odometry_frame>
-            <robot_base_frame>base_link</robot_base_frame>
+            <robot_base_frame>dummy</robot_base_frame>
             <publish_odom>true</publish_odom>
             <publish_odom_tf>true</publish_odom_tf>

File: description/lidar.xacro (robot description, xacro)
@@ -11,5 +11,5 @@
     </xacro:macro>
     <joint name="laser_joint" type="fixed">
-        <parent link="chassis"/>
+        <parent link="body_link"/>
         <child link="laser_frame"/>
         <origin xyz="0.122 0 0.212" rpy="0 0 0"/>
@@ -41,5 +41,5 @@
         <sensor name="laser" type="ray">
             <pose> 0 0 0 0 0 0 </pose>
-            <visualize>false</visualize>
+            <visualize>true</visualize>
             <update_rate>10</update_rate>
             <ray>

File: description/robot.urdf.xacro (robot description, xacro)
@@ -1,8 +1,22 @@
 <?xml version="1.0"?>
 <robot xmlns:xacro="http://www.ros.org/wiki/xacro"  name="robot">
-    <xacro:include filename="robot_core.xacro"/>
-    <!-- <xacro:include filename="ros2_control.xacro"/> -->
+    <!-- <xacro:include filename="robot_core.xacro"/>
+    <xacro:include filename="ros2_control.xacro"/> -->
     <!-- <xacro:include filename="roboclaw_ros2_control.xacro"/> -->
-    <xacro:include filename="gazebo_control.xacro"/>
-    <xacro:include filename="lidar.xacro"/>
+    <!-- <xacro:include filename="gazebo_control.xacro"/> -->
+    <!-- <xacro:include filename="lidar.xacro"/> -->
+    <!-- DIFF DRIVE GAZEBO -->
+    <!-- <xacro:include filename="robot_core.xacro"/>
+    <xacro:include filename="diff_dr_gaz.xacro"/> -->
+    <!-- SLAM STUFF -->
+    <xacro:arg name="use_ros2_control" default="true"/>
+    <xacro:arg name="sim_mode" default="false"/>
+    <xacro:include filename="robot_core.xacro" />
+    <xacro:if value="$(arg use_ros2_control)">
+        <xacro:include filename="ros2_control.xacro" />
+    </xacro:if>
+    <xacro:unless value="$(arg use_ros2_control)">
+        <xacro:include filename="gazebo_control.xacro" />
+    </xacro:unless>
+    <xacro:include filename="lidar.xacro" />
 </robot>

File: description/robot_core.xacro (robot description, xacro)
@@ -41,8 +41,8 @@
     </xacro:macro>
     <!-- Addin Gazebo Options -->
-    <link name="dummy">
+    <link name="base_link">
     </link>
     <joint name="base_footprint_joint" type="fixed">
-        <parent link="dummy" />
+        <parent link="base_link" />
         <child link="base_footprint" />
         <origin xyz ="0 0 0" rpy="0 0 0"/>
@@ -50,5 +50,5 @@
     <link name="base_footprint"></link>
     <joint name="body_joint" type="fixed">
-        <parent link="dummy" />
+        <parent link="base_link" />
         <child link="body_link" />
     </joint>
